File: headphone-amp.kicad_pcb (KiCad board)
At the start: 2 copper layers, 61.5 x 20 mm, 27 parts, among them J1 AudioJack4, J2 AudioJack4, J3 Conn_01x02_Male, SW1 SW_SPDT, U1 RC4580, U2 TMA0512D

Commit message: minor changes to filtering networks
Parts:
- C2, C9: value 10u -> 20u
- C5: value 100p -> 12n
- C6, C7: value 22p -> 402p
Changed lines of the file:
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@@
-(kicad_pcb (version 20171130) (host pcbnew 5.0.2-bee76a0~70~ubuntu18.04.1)
+(kicad_pcb (version 20171130) (host pcbnew "(5.0.2)-1")
   (general
     (thickness 1.6)
@@
       (effects (font (size 1 1) (thickness 0.15)))
     )
-    (fp_text value 10u (at 0 1.65 180) (layer F.Fab)
+    (fp_text value 20u (at 0 1.65 180) (layer F.Fab)
       (effects (font (size 1 1) (thickness 0.15)))
     )
@@
       (effects (font (size 1 1) (thickness 0.15)))
     )
-    (fp_text value 10u (at 0 1.65 180) (layer F.Fab)
+    (fp_text value 20u (at 0 1.65 180) (layer F.Fab)
       (effects (font (size 1 1) (thickness 0.15)))
     )
@@
       (effects (font (size 1 1) (thickness 0.15)))
     )
-    (fp_text value 22p (at 0 1.65 90) (layer F.Fab)
+    (fp_text value 402p (at 0 1.65 90) (layer F.Fab)
       (effects (font (size 1 1) (thickness 0.15)))
     )
@@
       (effects (font (size 1 1) (thickness 0.15)))
     )
-    (fp_text value 22p (at 0 1.65 270) (layer F.Fab)
+    (fp_text value 402p (at 0 1.65 270) (layer F.Fab)
       (effects (font (size 1 1) (thickness 0.15)))
     )
@@
       (effects (font (size 1 1) (thickness 0.15)))
     )
-    (fp_text value 100p (at 0 1.65 180) (layer F.Fab)
-      (effects (font (size 1 1) (thickness 0.15)))
-    )
+    (fp_text value 12n (at 0 1.65 180) (layer F.Fab)
+      (effects (font (size 1 1) (thickness 0.15)))
+    )

Commit message: added input filtering to DC-DC converter
Parts:
- added C10: 4u7, Capacitor_SMD:C_0805_2012Metric, F.Cu at (88.3, 91.2)
- added L3: 6u8, Inductor_SMD:L_0805_2012Metric, F.Cu at (89.2, 88.5)
Connections:
- SW1 pad 3: Net-(SW1-Pad3) -> Net-(C10-Pad1)
- U2 pad 1: Net-(SW1-Pad3) -> Net-(L3-Pad2)
Routing:
- net Net-(SW1-Pad3): track 35.6 -> 0.00 mm
- net Net-(C10-Pad1): track 0.00 -> 33.7 mm
- net Net-(L3-Pad2): track 0.00 -> 2.24 mm
- net Net-(C10-Pad2): track 22.7 -> 24.4 mm
Other:
- board text added: "5V Headphone Amplifier Designed by Joe Earlam Rev:"
- board text removed: "5V Headphone Amplifier Designed by Joe Earlam Rev: p1"

Commit message: Added input resistors
Parts:
- added R10: 10K, Resistor_SMD:R_0805_2012Metric, F.Cu at (135.8, 83.7)
- added R9: 10K, Resistor_SMD:R_0805_2012Metric, F.Cu at (132.3, 83.7)
Routing:
- net /Right_out: track 34.5 -> 38.8 mm
- net /Left_in: track 3.69 -> 6.41 mm
- net /Right_in: track 9.04 -> 11.5 mm
- net GND: vias 11 -> 12
Changed lines of the file:
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@@
     (thickness 1.6)
     (drawings 8)
-    (tracks 130)
+    (tracks 137)
     (zones 0)
-    (modules 29)
+    (modules 31)
     (nets 25)
   )
@@
   )
   (setup
-    (last_trace_width 0.25)
+    (last_trace_width 0.5)
     (user_trace_width 0.5)
     (trace_clearance 0.2)
@@
     (add_net "Net-(R8-Pad1)")
     (add_net "Net-(SW1-Pad1)")
+  )
+  (module Resistor_SMD:R_0805_2012Metric (layer F.Cu)
+    (at 135.763 83.693 180)
+    (descr "Resistor SMD 0805 (2012 Metric), square (rectangular) end terminal, IPC_7351 nominal, (Body size source: https://docs.google.com/spreadsheets/d/1BsfQQcO9C6DZCsRaXUlFlo91Tg2WpOkGARC1WS5S8t0/edit?usp=sharing), generated with kicad-footprint-generator")
+    (tags resistor)
+    (attr smd)
+    (fp_text reference R10 (at 2.921 1.524) (layer F.SilkS)
+      (effects (font (size 1 1) (thickness 0.15)))
+    )
+    (fp_text value 10K (at 0 1.65 180) (layer F.Fab)
+      (effects (font (size 1 1) (thickness 0.15)))
+    )
+    (fp_text user %R (at 0 0 180) (layer F.Fab)
+      (effects (font (size 0.5 0.5) (thickness 0.08)))
+    )
+    (fp_line (start 1.68 0.95) (end -1.68 0.95) (layer F.CrtYd) (width 0.05))
+    (fp_line (start 1.68 -0.95) (end 1.68 0.95) (layer F.CrtYd) (width 0.05))
+    (fp_line (start -1.68 -0.95) (end 1.68 -0.95) (layer F.CrtYd) (width 0.05))
+    (fp_line (start -1.68 0.95) (end -1.68 -0.95) (layer F.CrtYd) (width 0.05))
+    (fp_line (start -0.258578 0.71) (end 0.258578 0.71) (layer F.SilkS) (width 0.12))
+    (fp_line (start -0.258578 -0.71) (end 0.258578 -0.71) (layer F.SilkS) (width 0.12))
+    (fp_line (start 1 0.6) (end -1 0.6) (layer F.Fab) (width 0.1))
+    (fp_line (start 1 -0.6) (end 1 0.6) (layer F.Fab) (width 0.1))
+    (fp_line (start -1 -0.6) (end 1 -0.6) (layer F.Fab) (width 0.1))
+    (fp_line (start -1 0.6) (end -1 -0.6) (layer F.Fab) (width 0.1))
+    (pad 2 smd roundrect (at 0.9375 0 180) (size 0.975 1.4) (layers F.Cu F.Paste F.Mask) (roundrect_rratio 0.25)
+      (net 3 /Right_in))
+    (pad 1 smd roundrect (at -0.9375 0 180) (size 0.975 1.4) (layers F.Cu F.Paste F.Mask) (roundrect_rratio 0.25)
+      (net 5 GND))
+    (model ${KISYS3DMOD}/Resistor_SMD.3dshapes/R_0805_2012Metric.wrl
+      (at (xyz 0 0 0))
+      (scale (xyz 1 1 1))
+      (rotate (xyz 0 0 0))
+    )
+  )
+  (module Resistor_SMD:R_0805_2012Metric (layer F.Cu)
+    (at 132.334 83.693 180)
+    (descr "Resistor SMD 0805 (2012 Metric), square (rectangular) end terminal, IPC_7351 nominal, (Body size source: https://docs.google.com/spreadsheets/d/1BsfQQcO9C6DZCsRaXUlFlo91Tg2WpOkGARC1WS5S8t0/edit?usp=sharing), generated with kicad-footprint-generator")
+    (tags resistor)
+    (attr smd)
+    (fp_text reference R9 (at 2.921 1.27 270) (layer F.SilkS)
+      (effects (font (size 1 1) (thickness 0.15)))
+    )
+    (fp_text value 10K (at 0 1.65 180) (layer F.Fab)
+      (effects (font (size 1 1) (thickness 0.15)))
+    )
+    (fp_line (start -1 0.6) (end -1 -0.6) (layer F.Fab) (width 0.1))
+    (fp_line (start -1 -0.6) (end 1 -0.6) (layer F.Fab) (width 0.1))
+    (fp_line (start 1 -0.6) (end 1 0.6) (layer F.Fab) (width 0.1))
+    (fp_line (start 1 0.6) (end -1 0.6) (layer F.Fab) (width 0.1))
+    (fp_line (start -0.258578 -0.71) (end 0.258578 -0.71) (layer F.SilkS) (width 0.12))
+    (fp_line (start -0.258578 0.71) (end 0.258578 0.71) (layer F.SilkS) (width 0.12))
+    (fp_line (start -1.68 0.95) (end -1.68 -0.95) (layer F.CrtYd) (width 0.05))
+    (fp_line (start -1.68 -0.95) (end 1.68 -0.95) (layer F.CrtYd) (width 0.05))
+    (fp_line (start 1.68 -0.95) (end 1.68 0.95) (layer F.CrtYd) (width 0.05))
+    (fp_line (start 1.68 0.95) (end -1.68 0.95) (layer F.CrtYd) (width 0.05))
+    (fp_text user %R (at 0 0 180) (layer F.Fab)
+      (effects (font (size 0.5 0.5) (thickness 0.08)))
+    )
+    (pad 1 smd roundrect (at -0.9375 0 180) (size 0.975 1.4) (layers F.Cu F.Paste F.Mask) (roundrect_rratio 0.25)
+      (net 5 GND))
+    (pad 2 smd roundrect (at 0.9375 0 180) (size 0.975 1.4) (layers F.Cu F.Paste F.Mask) (roundrect_rratio 0.25)
+      (net 2 /Left_in))
+    (model ${KISYS3DMOD}/Resistor_SMD.3dshapes/R_0805_2012Metric.wrl
+      (at (xyz 0 0 0))
+      (scale (xyz 1 1 1))
+      (rotate (xyz 0 0 0))
+    )
   )
   (module Capacitor_SMD:C_0805_2012Metric (layer F.Cu)
@@
   (segment (start 127.7375 82.6) (end 128.5 82.6) (width 0.5) (layer F.Cu) (net 2))
   (segment (start 128.5 82.6) (end 129.899 81.201) (width 0.5) (layer F.Cu) (net 2))
+  (segment (start 130.85 83.1465) (end 131.3965 83.693) (width 0.5) (layer F.Cu) (net 2))
+  (segment (start 130.85 81.201) (end 130.85 83.1465) (width 0.5) (layer F.Cu) (net 2))
   (segment (start 127.7905 81.201) (end 127.7385 81.253) (width 0.5) (layer F.Cu) (net 3))
   (segment (start 127.7375 79.7625) (end 127.7375 80.7) (width 0.5) (layer F.Cu) (net 3))
@@
   (segment (start 123.081 80.7) (end 123.069 80.712) (width 0.5) (layer F.Cu) (net 4))
   (segment (start 125.8625 80.7) (end 123.081 80.7) (width 0.5) (layer F.Cu) (net 4))
-  (via (at 137.795 78.867) (size 0.8) (drill 0.4) (layers F.Cu B.Cu) (net 5))
   (via (at 137.922 88.773) (size 0.8) (drill 0.4) (layers F.Cu B.Cu) (net 5))
   (via (at 125.555 75.6285) (size 0.8) (drill 0.4) (layers F.Cu B.Cu) (net 5))
@@
   (via (at 98.298 91.821) (size 0.8) (drill 0.4) (layers F.Cu B.Cu) (net 5))
   (via (at 126.873 86.36) (size 0.8) (drill 0.4) (layers F.Cu B.Cu) (net 5))
-  (via (at 115.697 78.232) (size 0.8) (drill 0.4) (layers F.Cu B.Cu) (net 5))
+  (segment (start 134.85 83.6685) (end 134.8255 83.693) (width 0.5) (layer F.Cu) (net 3))
+  (segment (start 134.85 81.201) (end 134.85 83.6685) (width 0.5) (layer F.Cu) (net 3))
   (via (at 113.411 80.264) (size 0.8) (drill 0.4) (layers F.Cu B.Cu) (net 5))
+  (via (at 138.176 83.693) (size 0.8) (drill 0.4) (layers F.Cu B.Cu) (net 5))
+  (via (at 133.223 85.344) (size 0.8) (drill 0.4) (layers F.Cu B.Cu) (net 5))
+  (via (at 115.57 78.232) (size 0.8) (drill 0.4) (layers F.Cu B.Cu) (net 5))
   (segment (start 122.507 89.8375) (end 120.602 89.8375) (width 0.5) (layer F.Cu) (net 6))
   (segment (start 118.57 89.8375) (end 120.602 89.8375) (width 0.5) (layer F.Cu) (net 6))
@@
   (segment (start 121.745 76.977) (end 119.7765 76.977) (width 0.5) (layer F.Cu) (net 7))
   (segment (start 134.85 87.654) (end 134.85 91.234) (width 0.5) (layer F.Cu) (net 7))
-  (segment (start 136.271 86.233) (end 134.85 87.654) (width 0.5) (layer F.Cu) (net 7))
-  (segment (start 136.271 77.597) (end 136.271 86.233) (width 0.5) (layer F.Cu) (net 7))
-  (segment (start 134.874 76.2) (end 136.271 77.597) (width 0.5) (layer F.Cu) (net 7))
-  (segment (start 131.953 76.2) (end 134.874 76.2) (width 0.5) (layer F.Cu) (net 7))
+  (segment (start 135.128 87.376) (end 134.85 87.654) (width 0.5) (layer F.Cu) (net 7))
+  (segment (start 137.414 87.376) (end 135.128 87.376) (width 0.5) (layer F.Cu) (net 7))
+  (segment (start 139.573 85.217) (end 137.414 87.376) (width 0.5) (layer F.Cu) (net 7))
+  (segment (start 139.573 80.391) (end 139.573 85.217) (width 0.5) (layer F.Cu) (net 7))
+  (segment (start 135.382 76.2) (end 139.573 80.391) (width 0.5) (layer F.Cu) (net 7))
+  (segment (start 131.953 76.2) (end 135.382 76.2) (width 0.5) (layer F.Cu) (net 7))
+  (segment (start 123.65 75.184) (end 124.285 74.549) (width 0.5) (layer F.Cu) (net 7))
   (segment (start 123.65 76.977) (end 123.65 75.184) (width 0.5) (layer F.Cu) (net 7))
+  (segment (start 124.285 74.549) (end 126.238 74.549) (width 0.5) (layer F.Cu) (net 7))
   (segment (start 126.238 74.549) (end 128.397 76.708) (width 0.5) (layer F.Cu) (net 7))
   (segment (start 128.397 76.708) (end 131.445 76.708) (width 0.5) (layer F.Cu) (net 7))
   (segment (start 131.445 76.708) (end 131.953 76.2) (width 0.5) (layer F.Cu) (net 7))
-  (segment (start 124.285 74.549) (end 126.238 74.549) (width 0.5) (layer F.Cu) (net 7))
-  (segment (start 123.65 75.184) (end 124.285 74.549) (width 0.5) (layer F.Cu) (net 7))
   (segment (start 119.1775 80.7935) (end 119.259 80.712) (width 0.5) (layer F.Cu) (net 8))
   (segment (start 117.348 80.1435) (end 117.354 80.1375) (width 0.5) (layer F.Cu) (net 8))
